File: ROV_ECU_shield_nucleo/ROV_ECU_shield_nucleo.kicad_pcb (KiCad board)
At the start: 4 copper layers, 70 x 139.4 mm, 166 parts, among them IC1 DCL541A01, IC10 AP7375-33SA-7, IC11 MPU-6500, IC12 MPU-6500, IC13 MPU-6500, IC14 ATA6561-GAQW-N, IC15 AP7375-50SA-7, IC2 DCL541A01, IC3 DCL541A01, IC4 DCL541A01, IC5 DCL541A01, IC6 DCL541A01, IC7 ADUM3190TRQZ, IC8 ADUM3190TRQZ, IC9 DCL541A01, J1 24VPI, J10 ISO_AN2, J11 PWMO_4, J12 PWMO_5, J13 PWMO_6, J14 PWMI_1, J15 PWMI_2, J16 NMOS_SW1, J17 NMOS_SW2, J18 GPIO_2, J19 UART, J2 RS485_1, J20 I2C, J21 3.3VPO, J3 RS485_2, J4 CAN, J5 PWMO_1, J6 GPIO_1, J7 PWMO_2, J8 PWMO_3, J9 ISO_AN1, Q1 FDS6898A, U2 MAX3485, U3 MAX3485, U4 NUCLEOH723ZG, Y1 32.768k

Commit message: 試作完了．発注．
Parts:
- C50: moved to F.Cu
- moved C50 18.6 mm to (104.8, 70.0), turned to 90 degrees
Routing:
- net +24V: track 180.5 -> 172.5 mm
- net +3V3: track 410.2 -> 412.6 mm
- net GNDPWR: vias 42 -> 46
- net GND: vias 113 -> 119
Other:
- board text added: "ECU_SHIELD NUCLEO-H723ZG Ver.0.1.0"
