File: ROV_ECU_shield_nucleo/ROV_ECU_shield_nucleo.kicad_sch (KiCad schematic)
At the start: 120 parts, among them IC1 DCL541A01, IC2 DCL541A01, IC3 DCL541A01, IC4 DCL541A01, IC5 DCL541A01, IC6 DCL541A01, IC7 ADUM3190TRQZ, IC8 ADUM3190TRQZ, IC9 DCL541A01, J1 PWR_IN, J10 ISO_AN2, J11 PWMO_4, J12 PWMO_5, J13 PWMO_6, J14 PWMI_1, J15 PWMI_2, J16 LED1, J17 LED2, J2 RS485_1, J3 RS485_2, J4 RS485_2_TTL, J5 PWMO_1, J6 DIG_IO, J7 PWMO_2, J8 PWMO_3, J9 ISO_AN1, Q1 FDS6898A, U1 AZ1117-3.3, U2 MAX3485, U3 MAX3485, U4 NUCLEOH723ZG, U5 MAX3485

Commit message: 下記設計方針を定義．設計に反映． ・秋月電子での入手性を優先．（ZHコネクタ，LDO等） ・IMUは6軸（MPU6500は新規非推奨だが量産active） ・IMUメイン用途はレート制御・サブ用途が姿勢制御 ・2次側3.3V生成方法はひとまず秋月の高耐圧LDOとする．
設計TODO：
・ヒューズパッケージ未決定．
Parts:
- removed J6: DIG_IO, Connector_JST:JST_ZH_B8B-ZR_1x08_P1.50mm_Vertical, symbol Connector_Generic:Conn_01x08
- removed U1: AZ1117-3.3, Package_TO_SOT_SMD:SOT-223, symbol Regulator_Linear:AZ1117-3.3
- added C32, C36, C40: 2.2u, Capacitor_SMD:C_0603_1608Metric_Pad1.08x0.95mm_HandSolder, symbol Device:C_Small
- added C33, C34, C35, C37, C38, C39, C41, C42, C43: 0.1u, Capacitor_SMD:C_0603_1608Metric_Pad1.08x0.95mm_HandSolder, symbol Device:C_Small
- added D9: KDZVTR27B, Diode_SMD:D_SOD-123F, symbol Device:D_Zener
- added IC10: AP7375-33SA-7, SamacSys_Parts:SOT96P240X110-3N, symbol SamacSys_Parts:AP7375-33SA-7
- added IC11, IC12, IC13: MPU-6500, SamacSys_Parts:QFN40P300X300X95-25N-D, symbol SamacSys_Parts:MPU-6500
- added J18: GPIO_2, Connector_JST:JST_ZH_B6B-ZR_1x06_P1.50mm_Vertical, symbol Connector_Generic:Conn_01x06
- added J6: GPIO_1, Connector_JST:JST_ZH_B6B-ZR_1x06_P1.50mm_Vertical, symbol Connector_Generic:Conn_01x06
- added R43, R44, R45: 4.7k, Resistor_SMD:R_0603_1608Metric_Pad0.98x0.95mm_HandSolder, symbol Device:R
- C2: value 22u -> 1u
- C24, C29: value 0.1u -> TBD
- C3: value 22u -> 10u
- R25, R26, R27, R28, R29, R31, R32, R33, R34, R35: value 4.7k -> TBD
- R30, R36: value 470 -> TBD
Connections:
- net +24V: now also D9.1 (K), IC10.1 (VIN)
- net +3.3VP: now also IC10.2 (VOUT), J18.1 (Pin_1), J6.1 (Pin_1)
- net +3V3: now also C32.1, C33.1, C34.1, C36.1, C37.1, C38.1, C40.1, C41.1, C42.1, IC11.13 (VDD), IC11.8 (VDDIO), IC12.13 (VDD), IC12.8 (VDDIO), IC13.13 (VDD), IC13.8 (VDDIO), R43.1, R44.1, R45.1
- net GND: now also C32.2, C33.2, C34.2, C35.2, C36.2, C37.2, C38.2, C39.2, C40.2, C41.2, C42.2, C43.2, IC11.11 (FSYNC), IC11.18 (GND), IC11.20 (RESV_2), IC11.25 (T_PAD), IC12.11 (FSYNC), IC12.18 (GND), IC12.20 (RESV_2), IC12.25 (T_PAD), IC13.11 (FSYNC), IC13.18 (GND), IC13.20 (RESV_2), IC13.25 (T_PAD)
- net GNDPWR: now also D9.2 (A), IC10.3 (GND), J18.6 (Pin_6), J6.6 (Pin_6)
- net at D7.1 (CH1), IC4.14 (VO1): now also J6.2 (Pin_2)
- net at D7.3 (CH2), IC4.13 (VO2): now also J6.3 (Pin_3)
- net at D7.4 (CH3), IC4.12 (VO3): now also J6.4 (Pin_4)
- net at D7.6 (CH4), IC4.11 (VI4): now also J6.5 (Pin_5)
- net at D8.1 (CH1), IC6.14 (VO1): now also J18.2 (Pin_2)
- net at D8.3 (CH2), IC6.13 (VO2): now also J18.3 (Pin_3)
- net at D8.4 (CH3), IC6.12 (VO3): now also J18.4 (Pin_4)
- net at D8.6 (CH4), IC6.11 (VI4): now also J18.5 (Pin_5)
- new net: C35.1, IC11.10 (REGOUT)
- new net: C43.1, IC13.10 (REGOUT)
- new net: C39.1, IC12.10 (REGOUT)
- new net MISOA: IC11.9 (SDO/AD0), IC12.9 (SDO/AD0), IC13.9 (SDO/AD0)
- new net MOSIA: IC11.24 (SDA/SDI), IC12.24 (SDA/SDI), IC13.24 (SDA/SDI)
- new net RSPCKA: IC11.23 (SCL/SCLK), IC12.23 (SCL/SCLK), IC13.23 (SCL/SCLK)
- new net SSLA0: IC11.22 (NCS), IC12.22 (NCS), IC13.22 (NCS), R43.2, R44.2, R45.2
- no-connect marks 21 -> 35
Other:
- note added: "NOTE: --------------------------------- fc = foper/10 = (1/(2π)) * √(1/LC) --------------------------------- MIWI06 foper : 330kHz --------------------------------- https://edn.itmedia.co.jp/edn/articles/1809/25/news016.html ---------------------------------"
- note added: "Vin_max=45V Iout_max=300mA"
- note added: "絶縁ICを使ってみた(東京工業大学 ロボット技術研究会)"
- note removed: "NOTE: --------------------------------- fc = foper/10 = (1/(2π)) * √(1/LC) --------------------------------- MCWI03 foper : 300kHz --------------------------------- https://edn.itmedia.co.jp/edn/articles/1809/25/news016.html ---------------------------------"
- moved on the sheet: C2, C3, D1

Commit message: ・kicad ver. 10.05に変更． ・現在の設計でコミット． ・KiCad Routing Toolsプラグインをインストール．
Parts:
- added C44: 1000p, Capacitor_SMD:C_0603_1608Metric_Pad1.08x0.95mm_HandSolder, symbol Device:C_Small
- added D10: D1213A-04S-7, SamacSys_Parts:SOT65P210X110-6N, symbol SamacSys_Parts:D1213A-04S-7
- added J19: UART, Connector_JST:JST_ZH_B4B-ZR_1x04_P1.50mm_Vertical, symbol Connector_Generic:Conn_01x04
- added L2: L, Inductor_SMD:L_0603_1608Metric_Pad1.05x0.95mm_HandSolder, symbol Device:L
- added R46: 4.7k, Resistor_SMD:R_0603_1608Metric_Pad0.98x0.95mm_HandSolder, symbol Device:R
- added unit 1 of U4
- added unit 8 of U4
- added unit 7 of U4
- J16, J17: footprint Connector_JST:JST_XH_S2B-XH-A-1_1x02_P2.50mm_Horizontal -> Connector_JST:JST_XH_B2B-XH-A_1x02_P2.50mm_Vertical
Connections:
- net SPI1_MISO is gone; now on net PA6/SPI1_MISO: U4.CN7_12 (D12/SPI_A_MISO)
- net SPI1_MOSI is gone; now on net PB5/SPI1_MOSI: U4.CN7_14 (D11/SPI_A_MOSI/TIM_E_PWM1)
- net SPI1_SCK is gone; now on net PA5/SPI1_SCK: U4.CN7_10 (D13/SPI_A_SCK)
- net TIM2_CH4 is gone; now on net PB11/TIM2_CH4: U4.CN10_34 (D35/TIMER_C_PWM3)
- net +3V3: now also D10.5 (VP), J19.1 (Pin_1); no longer C21.1, C26.1, IC7.1 (VDD1), IC8.1 (VDD1), R27.2, R33.2
- net +5V: now also U4.CN11_6 (5V_EXT); no longer U4.CN8_9 (5V_CN8)
- net GND: now also U4.CN10_17 (GND_CN10__1), U4.CN10_22 (GND_CN10__2), U4.CN10_27 (GND_CN10__3), U4.CN10_5 (GND_CN10), U4.CN7_8 (GND_CN7), U4.CN8_11 (GND_CN8), U4.CN8_13 (GND_CN8__1), U4.CN9_12 (GND_CN9), U4.CN9_23 (GND_CN9__1), D10.2 (VN), J19.4 (Pin_4), R46.2, U4.CN3_1 (GND_CN3), U4.CN3_2 (GND_CN3__1), U4.CN4_1 (GND_CN4), U4.CN4_2 (GND_CN4__1); no longer C21.2, C23.1, C24.2, C26.2, C28.1, C29.2, IC7.2 (GND1_1), IC7.8 (GND1_2), IC8.2 (GND1_1), IC8.8 (GND1_2)
- net PG12/TIM23_CH1: now reaches IC4.3 (VI1)
- net PG12/TIM23_CH1: now also U4.CN10_2 (D7/IO)
- net PF7/TIM23_CH2: now reaches IC4.4 (VI2)
- net PF7/TIM23_CH2: now also U4.CN9_26 (D62/SAI_B_MCLK)
- net PG14/TIM23_CH3: now reaches IC4.5 (VI3)
- net PG14/TIM23_CH3: now also U4.CN10_12 (D2/IO)
- net PE6/TIM15_CH2: now reaches IC4.6 (VO4)
- net PE6/TIM15_CH2: now also U4.CN10_28 (D38/TIMER_A_BKIN2)
- net PE12/D39: now reaches IC2.4 (VI2)
- net PE12/D39: now also U4.CN10_26 (D39/TIMER_A_PWM3N)
- net PE10/D40: now reaches IC2.5 (VI3)
- net PE10/D40: now also U4.CN10_24 (D40/TIMER_A_PWM2N)
- net at IC9.13 (VO2): now also R41.1; no longer R39.1
- net at IC9.14 (VO1): now also R39.1; no longer R41.1
- net PC8/TIM3_CH3: now reaches IC9.3 (VI1)
- net PC8/TIM3_CH3: now also U4.CN8_2 (D43/SDMMC_D0)
- net PC9/TIM3_CH4: now reaches IC9.4 (VI2)
- net PC9/TIM3_CH4: now also U4.CN8_4 (D44/SDMMC_D1/I2S_A_CKIN)
- net PC6/USART6_TX: now reaches U4.CN7_1 (D16/I2S_A_MCK)
- net PC6/USART6_TX: now also D10.4 (CH3), J19.2 (Pin_2)
- net PC7/USART6_RX: now reaches U4.CN7_11 (D21/I2S_B_MCK)
- net PC7/USART6_RX: now also D10.6 (CH4), J19.3 (Pin_3), R46.1
- net PF3/TIM23_CH4: now reaches U4.CN7_20 (D8/IO)
- net PF3/TIM23_CH4: now also IC6.3 (VI1)
- net PE15/D37: now reaches IC1.4 (VI2)
- net PE15/D37: now also U4.CN10_30 (D37/TIMER_A_BKIN1)
- net PG2/D49: now reaches U4.CN8_14 (D49/IO)
- net PG2/D49: now also IC13.22 (NCS), R45.2
- net PG3/D50: now reaches U4.CN8_16 (D50/IO)
- net PD0/D67/FDCAN1_RX: now reaches U4.CN9_25 (D67/CAN_RX)
- net PD0/D67/FDCAN1_RX: now also IC6.6 (VO4)
- net PD1/D66/FDCAN1_TX: now reaches U4.CN9_27 (D66/CAN_TX)
- net PD1/D66/FDCAN1_TX: now also IC6.5 (VI3)
- net PF9/TIM14_CH1: now reaches U4.CN9_28 (D63/SAI_B_FS)
- net PF9/TIM14_CH1: now also IC6.4 (VI2)
- net PG0/D65: now reaches U4.CN9_29 (D65/IO)
- net PG1/D64: now reaches U4.CN9_30 (D64/IO)
- net at U4.CN10_1 (AVDD): now also L2.1
- net PE8/D42: now reaches U4.CN10_18 (D42/TIMER_A_PWM1N)
- net PE8/D42: now also IC12.22 (NCS), R44.2
- net PE7/D41: now reaches U4.CN10_20 (D41/TIMER_A_ETR)
- net PE7/D41: now also IC11.22 (NCS), R43.2
- net GNDA: now reaches U4.CN10_3 (AGND_CN10)
- net GNDA: now also C21.2, C23.1, C24.2, C26.2, C28.1, C29.2, IC7.2 (GND1_1), IC7.8 (GND1_2), IC8.2 (GND1_1), IC8.8 (GND1_2), C44.2
- net ADC1_INP10 renamed PC0/ADC1_INP10
- net ADC1_INP15 renamed PA3/ADC1_INP15
- net ADC1_INP5: no longer names the net of U4.CN9_7 (A3/ADC12_INP5)
- net ADC3_INP0: no longer names the net of U4.CN9_9 (A4/ADC123_INP12/I2C1_SDA)
- net ADC3_INP1: no longer names the net of U4.CN9_5 (A2/ADC12_INP13)
- net ADC3_INP6: no longer names the net of U4.CN9_11 (A5/ADC3_INP6/I2C1_SCL)
- net MISOA renamed PA6/SPI1_MISO
- net MOSIA renamed PB5/SPI1_MOSI
- net RSPCKA renamed PA5/SPI1_SCK
- removed net SSLA0: IC11.22 (NCS), IC12.22 (NCS), IC13.22 (NCS), R43.2, R44.2, R45.2
- net TIM1_CH1 renamed PE9/TIM1_CH1
- net TIM1_CH2 renamed PE11/TIM1_CH2
- net TIM1_CH3 renamed PE13/TIM1_CH3
- net TIM1_CH4 renamed PA0/TIM2_CH1
- net PA0/TIM2_CH1: now also U4.CN10_29 (D32/TIMER_C_PWM1); no longer U4.CN10_8 (D4/IO)
- net TIM2_CH1 renamed PB10/TIM2_CH3
- net PB10/TIM2_CH3: now also U4.CN10_32 (D36/TIMER_C_PWM2); no longer U4.CN10_29 (D32/TIMER_C_PWM1)
- net TIM2_CH3 renamed PB11/TIM2_CH4
- net PB11/TIM2_CH4: no longer U4.CN10_32 (D36/TIMER_C_PWM2)
- net TIM4_CH3 renamed PD14/TIM4_CH3
- net TIM4_CH4 renamed PD15/TIM4_CH4
- net USART1_RX renamed PB7/USART1_RX
- net USART1_TX renamed PB6/USART1_TX
- net USART2_RX renamed PD6/USART2_RX
- net USART2_TX renamed PD5/USART2_TX
- new net +3.3VA: C21.1, C26.1, C44.1, IC7.1 (VDD1), IC8.1 (VDD1), L2.2, R27.2, R33.2
- new net PE14/TIM1_CH4: U4.CN10_8 (D4/IO)
- no-connect marks 35 -> 157
Other:
- note added: "reserved:LD1"
- moved on the sheet: C10, C14, C15, C18, C19, C21, C26, C30, C31, C32, C33, C34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

Commit message: 更新
Parts:
- removed F1, F2: 5A, symbol Device:Fuse
- removed R19: 120, Resistor_SMD:R_0603_1608Metric_Pad0.98x0.95mm_HandSolder, symbol Device:R
- removed R20: 10, Resistor_SMD:R_0603_1608Metric_Pad0.98x0.95mm_HandSolder, symbol Device:R
- removed R21: 1k, Resistor_SMD:R_0603_1608Metric_Pad0.98x0.95mm_HandSolder, symbol Device:R
- removed R22, R23, R24: 4.7k, Resistor_SMD:R_0603_1608Metric_Pad0.98x0.95mm_HandSolder, symbol Device:R
- removed U5: MAX3485, Package_SO:SOIC-8_3.9x4.9mm_P1.27mm, symbol Interface_UART:MAX3485
- added AC1: BNO085, SamacSys_Parts:BNO085, symbol SamacSys_Parts:BNO085
- added C45, C46, C47: 0.1u, Capacitor_SMD:C_0603_1608Metric_Pad1.08x0.95mm_HandSolder, symbol Device:C_Small
- added C48: 10u, Capacitor_SMD:C_0603_1608Metric_Pad1.08x0.95mm_HandSolder, symbol Device:C_Small
- added D11: D, Diode_SMD:D_SOD-323_HandSoldering, symbol Device:D
- added IC14: ATA6561-GAQW-N, SamacSys_Parts:SOIC127P600X175-8N, symbol SamacSys_Parts:ATA6561-GAQW-N
- added IC15: AP7375-50SA-7, SamacSys_Parts:SOT96P240X110-3N, symbol SamacSys_Parts:AP7375-33SA-7
- added J20: I2C, Connector_JST:JST_ZH_B4B-ZR_1x04_P1.50mm_Vertical, symbol Connector_Generic:Conn_01x04
- added J21: 3.3VPO, Connector_JST:JST_ZH_B2B-ZR_1x02_P1.50mm_Vertical, symbol Connector_Generic:Conn_01x02
- added R47, R48, R49, R50, R51, R52, R53, R54: 4.7k, Resistor_SMD:R_0603_1608Metric_Pad0.98x0.95mm_HandSolder, symbol Device:R
- C11: value 0.1u -> 1u
- C44: value 1000p -> 0.1u
- F3: footprint (none) -> Fuse:Fuseholder_Blade_Mini_Keystone_3568
- J1: value PWR_IN -> 24VPI; footprint Connector_JST:JST_XH_S2B-XH-A-1_1x02_P2.50mm_Horizontal -> Connector_JST:JST_ZH_B2B-ZR_1x02_P1.50mm_Vertical
- J16: value LED1 -> NMOS_SW1; footprint Connector_JST:JST_XH_B2B-XH-A_1x02_P2.50mm_Vertical -> Connector_JST:JST_ZH_B2B-ZR_1x02_P1.50mm_Vertical
- J17: value LED2 -> NMOS_SW2; footprint Connector_JST:JST_XH_B2B-XH-A_1x02_P2.50mm_Vertical -> Connector_JST:JST_ZH_B2B-ZR_1x02_P1.50mm_Vertical
- J4: value RS485_2_TTL -> CAN
- R17: value 1k -> 60
- R18: value 10 -> 60
Connections:
- net +24V: now also C11.1, J16.1 (Pin_1), J17.1 (Pin_1), D11.1 (K), IC15.1 (VIN)
- net +3.3VP: now also C46.1, IC14.5 (VIO), J21.1 (Pin_1); no longer C11.1, D3.5 (VP), J4.1 (Pin_1), R17.1
- net +3V3: now also J20.1 (Pin_1), R53.1, R54.1
- net GND: now also J20.4 (Pin_4), R47.2, R48.2, R49.2, R50.2, R51.2, R52.2
- net GNDPWR: now also C45.2, C46.2, C47.2, C48.2, IC14.2 (GND), IC15.3 (GND), J21.2 (Pin_2)
- net PA5/SPI1_SCK: now also U4.CN7_2 (D15/I2C_A_SCL); no longer IC12.23 (SCL/SCLK), IC13.23 (SCL/SCLK), U4.CN7_10 (D13/SPI_A_SCK)
- net PA6/SPI1_MISO: no longer IC12.9 (SDO/AD0), IC13.9 (SDO/AD0)
- net PB5/SPI1_MOSI: no longer IC12.24 (SDA/SDI), IC13.24 (SDA/SDI)
- net PB7/USART1_RX: now also R52.1
- net PD0/D67/FDCAN1_RX: now also R48.1
- net PD14/TIM4_CH3: now also R49.1
- net PD15/TIM4_CH4: now also R50.1
- net PD6/USART2_RX: now also R51.1
- net PE6/TIM15_CH2: now also R47.1
- net at R18.1: now also D3.3 (CH2), J4.2 (Pin_2), IC14.6 (CANL)
- net at R17.2: now also D3.1 (CH1), J4.3 (Pin_3), IC14.7 (CANH)
- net at D2.1 (CH1), J2.2 (Pin_2), R2.2: no longer R18.2
- net at IC9.13 (VO2): now also R39.1; no longer R41.1
- net at IC9.14 (VO1): now also R41.1; no longer R39.1
- net PB3/SPI3_SCK: now reaches U4.CN7_15 (D23/I2S_B_CK/SPI_B_SCK)
- net PB3/SPI3_SCK: now also IC13.23 (SCL/SCLK)
- net PB4/SPI3_MISO: now reaches U4.CN7_19 (D25/SPI_B_MISO)
- net PB4/SPI3_MISO: now also IC13.9 (SDO/AD0)
- net PB9/I2C1_SDA: now reaches U4.CN7_4 (D14/I2C_A_SDA)
- net PB9/I2C1_SDA: now also D10.1 (CH1), J20.2 (Pin_2), R53.2
- net PC12/SPI3_MOSI: now reaches U4.CN8_10 (D47/SDMMC_CK)
- net PC12/SPI3_MOSI: now also IC13.24 (SDA/SDI)
- net CANBUS_STBY: now reaches D8.3 (CH2), IC6.13 (VO2), J18.3 (Pin_3)
- net CANBUS_STBY: now also IC14.8 (STBY)
- net CANBUS_TX: now reaches D8.4 (CH3), IC6.12 (VO3), J18.4 (Pin_4)
- net CANBUS_TX: now also IC14.1 (TXD)
- net CANBUS_RX: now reaches D8.6 (CH4), IC6.11 (VI4), J18.5 (Pin_5)
- net CANBUS_RX: now also IC14.4 (RXD)
- net at D3.4 (CH3): no longer J4.2 (Pin_2)
- net at D3.6 (CH4): no longer J4.3 (Pin_3)
- net PC3/SPI2_MOSI: now reaches U4.CN9_5 (A2/ADC12_INP13)
- net PC3/SPI2_MOSI: now also IC12.24 (SDA/SDI)
- net PD3/SPI2_SCK: now reaches U4.CN9_8 (D54/USART_B_RTS)
- net PD3/SPI2_SCK: now also IC12.23 (SCL/SCLK)
- net PC2/SPI2_MISO: now reaches U4.CN9_9 (A4/ADC123_INP12/I2C1_SDA)
- net PC2/SPI2_MISO: now also IC12.9 (SDO/AD0)
- net PB8/I2C1_SCL: now reaches D10.3 (CH2)
- net PB8/I2C1_SCL: now also U4.CN7_10 (D13/SPI_A_SCK), J20.3 (Pin_3), R54.2
- net PE10/D40: no longer names the net of IC2.5 (VI3)
- net PE10/D40: no longer U4.CN10_24 (D40/TIMER_A_PWM2N)
- net UART_BUS2_DEV_EN: no longer names the net of IC2.12 (VO3)
- new net: C45.1, R17.1, R18.2
- new net +5VP: C47.1, C48.1, D11.2 (A), D3.5 (VP), IC14.3 (VCC), IC15.2 (VOUT), J4.1 (Pin_1)
- no-connect marks 157 -> 150
Other:
- note added: "AP7375-**SA Vin_max=45V Iout_max=300mA"
- note added: "スラスタ用PWM出力 x6 センサ用RS485バス x1 スラスタ用RS485バス x1 ライト制御用FET駆動 x2 センサ/RC制御用PWM入力 x2 汎用センサ用AN入力x 1 水圧センサ用AN入力x 1 その他デジタルGPI x その他デジタルGPO x"
- note removed: "Vin_max=45V Iout_max=300mA"
- note removed: "スラスタ用PWM出力 x6 センサ用RS485バス x1 スラスタ用RS485バス x1 ライト制御用FET駆動 x2 センサ/RC制御用PWM入力 x3 電流センサ用AN入力x 1 水圧センサ用AN入力x 1 その他デジタルGPI x その他デジタルGPO x GPS用RS485変換付き入力ポート x1"
- moved on the sheet: C1, C10, C12, C13, C14, C15, C16, C17, C18, C19, C2, C20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

Commit message: ・sch 誤接続修正（I2C1_SCL/SPI1_SCK）修正． ・BNO085 H_INTN端子を外部割込み端子へ接続． ・A/Wレイアウトブラッシュアップ．
Parts:
- added C49, C51, C52: 0.1u, Capacitor_SMD:C_0603_1608Metric_Pad1.08x0.95mm_HandSolder, symbol Device:C_Small
- added C50: 4.7u, Capacitor_SMD:C_1206_3216Metric_Pad1.33x1.80mm_HandSolder, symbol Device:C_Small
- added C54, C55: 22p, Capacitor_SMD:C_0603_1608Metric_Pad1.08x0.95mm_HandSolder, symbol Device:C_Small
- added JP3: SolderJumper_3_Open, Jumper:SolderJumper-3_P1.3mm_Open_RoundedPad1.0x1.5mm, symbol Jumper:SolderJumper_3_Open
- added R55, R56: 10k, Resistor_SMD:R_0603_1608Metric_Pad0.98x0.95mm_HandSolder, symbol Device:R
- added TP1, TP2: TestPoint, TestPoint:TestPoint_Pad_D1.0mm, symbol Connector:TestPoint
- added Y1: 32.768k, Crystal:Crystal_SMD_3215-2Pin_3.2x1.5mm, symbol Device:Crystal
Connections:
- net PE14/TIM1_CH4 is gone; now on net PE14/EXTI14: U4.CN10_8 (D4/IO)
- net +3V3: now also AC1.28 (VDDIO), AC1.3 (VDD), C49.1, C50.1, C52.1, JP3.1 (A), R55.1, R56.1
- net GND: now also AC1.2 (GND_1), AC1.25 (GND_2), AC1.5 (PS1), AC1.6 (PS0/WAKE), C49.2, C50.2, C51.1, C52.2, C54.1, C55.1, JP3.3 (B)
- net PA5/SPI1_SCK: now also U4.CN7_10 (D13/SPI_A_SCK); no longer U4.CN7_2 (D15/I2C_A_SCL)
- net PB8/I2C1_SCL: now also AC1.19 (H_SCL/SCK/RX), U4.CN7_2 (D15/I2C_A_SCL); no longer U4.CN7_10 (D13/SPI_A_SCK)
- net PB9/I2C1_SDA: now also AC1.20 (H_SDA/H_MISO/TX)
- net nRST: now reaches U4.CN8_5 (NRST_CN8)
- net nRST: now also AC1.11 (NRST), R56.2
- net at AC1.10 (CLKSEL0): now also R55.2, TP1.1
- net PE14/EXTI14: now reaches AC1.14 (H_INTN)
- net at AC1.17 (SA0/H_MOSI): now also JP3.2 (C)
- net at AC1.26 (XOUT32/CLKSEL1): now also C55.2, Y1.2
- net at AC1.27 (XIN32): now also C54.2, Y1.1
- net at AC1.4 (BOOTN): now also TP2.1
- net at AC1.9 (CAP): now also C51.2
- no-connect marks 150 -> 161
Other:
- note added: "FC-135 32.768000KHz 12.5 +20.0-20.0 (F)"
- moved on the sheet: C45, R17, R18
